Commit message: Added updated ReadMe file and updated URDF for compatibility with Minshen's realsense code

File: xarm_description/urdf/xarm6.urdf.xacro (robot description, xacro)
@@ -328,4 +328,17 @@
       link="${prefix}link_eef" />
   </joint>
+  <link name="${prefix}cam_link">
+    </link>
+  <joint
+    name="${prefix}joint_cam"
+    type="fixed">
+    <origin
+      xyz="0.07 -0.04 0.03"
+      rpy="0 0 1.5708" />
+    <parent
+      link="${prefix}link_eef" />
+    <child
+      link="${prefix}cam_link" />
+  </joint>
   </xacro:macro>
 </robot>
