Commit message: Implementing mobile base and bin urdf models

File: xarm_description/urdf/xarm6_robot_macro.xacro (robot description, xacro)
@@ -56,4 +56,56 @@
       />
     </xacro:if>
+        <!-- Additional Base and Trash Bin for the xArm -->
+    <joint name="base_joint" type="fixed">
+      <origin xyz="-0.13 0 0" rpy="0 0 0"/>
+      <parent link="world"/>
+      <child link="base_link"/>
+    </joint>
+    <link name="base_link">
+      <visual>
+        <origin xyz="0 0 0.186" rpy="0 0 0"/>
+        <geometry>
+          <box size="0.46 0.38 0.372"/>
+        </geometry>
+        <material name="Red"/>
+      </visual>
+      <collision>
+        <origin xyz="0 0 0.186" rpy="0 0 0"/>
+        <geometry>
+          <box size="0.46 0.38 0.372"/>
+        </geometry>
+      </collision>
+      <inertial>
+          <origin xyz="0 0 0.186" rpy="0 0 0"/>
+          <mass value="12" />
+          <inertia ixx="2.26" ixy="0.0" ixz="0.0" iyy="6.26" iyz="0.0" izz="8.5" />
+      </inertial>
+    </link>
+    <joint name="bin_joint" type="fixed">
+      <origin xyz="-0.305 0 0.222" rpy="0 0 0"/>
+      <parent link="base_link"/>
+      <child link="bin_link"/>
+    </joint>
+    <link name="bin_link">
+      <visual>
+        <origin xyz="0 0 0.075" rpy="0 0 0"/>
+        <geometry>
+          <box size="0.15 0.26 0.15"/>
+        </geometry>
+        <material name="Silver"/>
+      </visual>
+      <collision>
+        <origin xyz="0 0 0.075" rpy="0 0 0"/>
+        <geometry>
+          <box size="0.15 0.26 0.15"/>
+        </geometry>
+      </collision>
+      <inertial>
+          <origin xyz="0 0 0.186" rpy="0 0 0"/>
+          <mass value="12" />
+          <inertia ixx="2.26" ixy="0.0" ixz="0.0" iyy="6.26" iyz="0.0" izz="8.5" />
+      </inertial>
+    </link>
+    <!-- End of additions -->
   </xacro:macro>
 </robot>

File: xarm_description/urdf/xarm6_with_gripper.xacro (robot description, xacro)
@@ -7,5 +7,5 @@
   <xacro:arg name="velocity_control" default="false"/>
   <!-- To add realsense d435i and gripper, set 'add_realsense_d435i' = true -->
-  <xacro:arg name="add_realsense_d435i" default="false"/>
+  <xacro:arg name="add_realsense_d435i" default="true"/>
   <xacro:arg name="use_gazebo_camera" default="false"/>
   <!-- load xarm6 robot -->

Commit message: added modified bin attachment

File: xarm_description/urdf/xarm6_robot_macro.xacro (robot description, xacro)
@@ -89,14 +89,14 @@
     <link name="bin_link">
       <visual>
-        <origin xyz="0 0 0.075" rpy="0 0 0"/>
+        <origin xyz="0 0 0.155" rpy="0 0 0"/>
         <geometry>
-          <box size="0.15 0.26 0.15"/>
+          <box size="0.15 0.33 0.31"/>
         </geometry>
         <material name="Silver"/>
       </visual>
       <collision>
-        <origin xyz="0 0 0.075" rpy="0 0 0"/>
+        <origin xyz="0 0 0.155" rpy="0 0 0"/>
         <geometry>
-          <box size="0.15 0.26 0.15"/>
+          <box size="0.15 0.33 0.31"/>
         </geometry>
       </collision>

Commit message: able to halt the BZ

File: xarm_description/urdf/xarm6_robot_macro.xacro (robot description, xacro)
@@ -60,7 +60,7 @@
       <origin xyz="-0.13 0 0" rpy="0 0 0"/>
       <parent link="world"/>
-      <child link="base_link"/>
+      <child link="base_link_2"/>
     </joint>
-    <link name="base_link">
+    <link name="base_link_2">
       <visual>
         <origin xyz="0 0 0.186" rpy="0 0 0"/>
@@ -84,5 +84,5 @@
     <joint name="bin_joint" type="fixed">
       <origin xyz="-0.305 0 0.222" rpy="0 0 0"/>
-      <parent link="base_link"/>
+      <parent link="base_link_2"/>
       <child link="bin_link"/>
     </joint>
